File: Christmas Ornament 2024.kicad_sch (KiCad schematic)
At the start: 34 parts, among them J1 USB_B_Micro, J2 Conn_01x03, J3 Conn_01x02, J4 Conn_01x03, U1 RP2040, U2 LIS3DH, U3 AMS1117-3.3, U4 W25Q128JVS, U5 TLV61070ADBV, Y1 Crystal

Commit message: Add LEDs and resistors
Parts:
- added D2: Red LED, LED_SMD:LED_0805_2012Metric_Pad1.15x1.40mm_HandSolder, symbol Device:LED_Small
- added R5: 100, symbol Device:R_Small
- D1: value LED_Small -> Green LED; footprint (none) -> LED_SMD:LED_0805_2012Metric_Pad1.15x1.40mm_HandSolder; JLCPCB PN (none) -> C2297
Other:
- note added: "R1"
- note added: "R1 = (Vout/Vref - 1) * R2 112800 = (5.2/0.5 - 1) x 12000"
- note added: "R2"
Changed lines of the file:
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@@
 		)
 	)
+	(text "R1 = (Vout/Vref - 1) * R2\n112800 = (5.2/0.5 - 1) x 12000"
+		(exclude_from_sim no)
+		(at 213.106 120.904 0)
+		(effects
+			(font
+				(size 1.27 1.27)
+			)
+		)
+	)
+	(text "R1"
+		(exclude_from_sim no)
+		(at 208.28 104.394 90)
+		(effects
+			(font
+				(size 1.27 1.27)
+			)
+		)
+	)
+	(text "R2"
+		(exclude_from_sim no)
+		(at 208.28 113.538 90)
+		(effects
+			(font
+				(size 1.27 1.27)
+			)
+		)
+	)
 	(global_label "SWD"
 		(shape input)
@@
 	)
 	(symbol
+		(lib_id "Device:LED_Small")
+		(at 160.02 69.85 180)
+		(unit 1)
+		(exclude_from_sim no)
+		(in_bom yes)
+		(on_board yes)
+		(dnp no)
+		(fields_autoplaced yes)
+		(property "Reference" "D2"
+			(at 159.9565 63.5 0)
+			(effects
+				(font
+					(size 1.27 1.27)
+				)
+			)
+		)
+		(property "Value" "Red LED"
+			(at 159.9565 66.04 0)
+			(effects
+				(font
+					(size 1.27 1.27)
+				)
+			)
+		)
+		(property "Footprint" "LED_SMD:LED_0805_2012Metric_Pad1.15x1.40mm_HandSolder"
+			(at 160.02 69.85 90)
+			(effects
+				(font
+					(size 1.27 1.27)
+				)
+				(hide yes)
+			)
+		)
+		(property "Datasheet" "~"
+			(at 160.02 69.85 90)
+			(effects
+				(font
+					(size 1.27 1.27)
+				)
+				(hide yes)
+			)
+		)
+		(property "Description" "LED Red, 0805"
+			(at 160.02 69.85 0)
+			(effects
+				(font
+					(size 1.27 1.27)
+				)
+				(hide yes)
+			)
+		)
+		(property "JLCPCB PN" "C2296"
+			(at 160.02 69.85 0)
+			(effects
+				(font
+					(size 1.27 1.27)
+				)
+				(hide yes)
+			)
+		)
+		(pin "2"
+		)
+		(pin "1"
+		)
+		(instances
+			(project "Christmas Ornament 2024"
+				(path "/3b6a41c6-a8dd-4eec-bbf2-75fca69ae903"
+					(reference "D2")
+					(unit 1)
+				)
+			)
+		)
+	)
+	(symbol
 		(lib_id "power:+3V3")
 		(at 255.27 124.46 0)
@@
 	)
 	(symbol
+		(lib_id "Device:R_Small")
+		(at 148.59 58.42 90)
+		(unit 1)
+		(exclude_from_sim no)
+		(in_bom yes)
+		(on_board yes)
+		(dnp no)
+		(fields_autoplaced yes)
+		(property "Reference" "R5"
+			(at 148.59 53.34 90)
+			(effects
+				(font
+					(size 1.27 1.27)
+				)
+			)
+		)
+		(property "Value" "100"
+			(at 148.59 55.88 90)
+			(effects
+				(font
+					(size 1.27 1.27)
+				)
+			)
+		)
+		(property "Footprint" ""
+			(at 148.59 58.42 0)
+			(effects
+				(font
+					(size 1.27 1.27)
+				)
+				(hide yes)
+			)
+		)
+		(property "Datasheet" "~"
+			(at 148.59 58.42 0)
+			(effects
+				(font
+					(size 1.27 1.27)
+				)
+				(hide yes)
+			)
+		)
+		(property "Description" "Resistor, small symbol"
+			(at 148.59 58.42 0)
+			(effects
+				(font
+					(size 1.27 1.27)
+				)
+				(hide yes)
+			)
+		)
+		(property "JLCPCB PN" "C17408"
+			(at 148.59 58.42 0)
+			(effects
+				(font
+					(size 1.27 1.27)
+				)
+				(hide yes)
+			)
+		)
+		(pin "2"
+		)
+		(pin "1"
+		)
+		(instances
+			(project ""
+				(path "/3b6a41c6-a8dd-4eec-bbf2-75fca69ae903"
+					(reference "R5")
+					(unit 1)
+				)
+			)
+		)
+	)
+	(symbol
 		(lib_id "power:GND")
 		(at 109.22 148.59 0)
@@
 			)
 		)
-		(property "Value" "LED_Small"
+		(property "Value" "Green LED"
 			(at 159.9565 54.61 0)
 			(effects
@@
 			)
 		)
-		(property "Footprint" ""
+		(property "Footprint" "LED_SMD:LED_0805_2012Metric_Pad1.15x1.40mm_HandSolder"
 			(at 160.02 58.42 90)
 			(effects
@@
 			)
 		)
-		(property "Description" "Light emitting diode, small symbol"
+		(property "Description" "LED Green, 0805"
 			(at 160.02 58.42 0)
 			(effects
@@
 			)
 		)
-		(property "JLCPCB PN" ""
+		(property "JLCPCB PN" "C2297"
 			(at 160.02 58.42 0)
 			(effects

Commit message: Schematic Finished
Parts:
- removed J3: Conn_01x02, Connector_PinHeader_2.54mm:PinHeader_1x02_P2.54mm_Vertical, symbol Connector_Generic:Conn_01x02
- added C19, C20, C22: 1u, Capacitor_SMD:C_0402_1005Metric_Pad0.74x0.62mm_HandSolder, symbol Device:C_Small
- added C21: 680p, Capacitor_SMD:C_0603_1608Metric, symbol Device:C_Small
- added D10, D11, D12, D3, D5, D6, D9: Green LED, LED_SMD:LED_0805_2012Metric_Pad1.15x1.40mm_HandSolder, symbol Device:LED_Small
- added D13, D14, D15, D16, D17, D4, D7, D8: Red LED, LED_SMD:LED_0805_2012Metric_Pad1.15x1.40mm_HandSolder, symbol Device:LED_Small
- added J3, J5: Conn_01x03, Connector_PinHeader_2.54mm:PinHeader_1x03_P2.54mm_Vertical, symbol Connector_Generic:Conn_01x03
- added JP1: Jumper_2_Open, Jumper:SolderJumper-2_P1.3mm_Open_RoundedPad1.0x1.5mm, symbol Jumper:Jumper_2_Open
- added R10, R11, R12, R13, R14, R15, R16, R17, R18, R19, R20, R21, R22, R23, R7, R8, R9: 100, Resistor_SMD:R_0805_2012Metric_Pad1.20x1.40mm_HandSolder, symbol Device:R_Small
- added R6: 10k, Resistor_SMD:R_0805_2012Metric_Pad1.20x1.40mm_HandSolder, symbol Device:R_Small
- added SW1, SW2, SW3, SW4: PTS815, ChristmasOrnamentFootprints:PTS815 Series, symbol Switch:SW_MEC_5E
- added U6: TMP235, Package_TO_SOT_SMD:SOT-353_SC-70-5, symbol ChristmasOrnamentSymbols:TMP235
- J2: JLCPCB PN (none) -> DNP
- J4: JLCPCB PN (none) -> C49257
- R5: footprint (none) -> Resistor_SMD:R_0805_2012Metric_Pad1.20x1.40mm_HandSolder
Connections:
- net I2C_SCL is gone; now on net I2C SCL: U2.4 (SPC)
- net I2C_SDA is gone; now on net I2C SDA: U2.6 (SDI)
- net +3V3: now also C19.1, C20.1, R6.2, R8.2, SW1.1, SW1.2
- net +BATT: now also J5.1 (Pin_1)
- net GND: now also D1.1 (K), D2.1 (K), U1.19 (TESTEN), C19.2, C20.2, C21.2, C22.2, D10.1 (K), D11.1 (K), D12.1 (K), D13.1 (K), D14.1 (K), D15.1 (K), D16.1 (K), D17.1 (K), D3.1 (K), D4.1 (K), D5.1 (K), D6.1 (K), D7.1 (K), D8.1 (K), D9.1 (K), J3.2 (Pin_2), J5.3 (Pin_3), JP1.1 (A), SW2.3 (K), SW2.4 (A), SW3.3 (K), SW3.4 (A), SW4.3 (K), SW4.4 (A), U6.2 (GND); no longer U2.7 (SDO)
- net QSPI SS: now also R6.1, SW2.1, SW2.2
- net LED SW: now reaches U1.11 (GPIO8)
- net LED SW: now also R12.1
- net LED SSW: now reaches U1.12 (GPIO9)
- net LED SSW: now also R14.1
- net LIS3DH INT1: now reaches U1.13 (GPIO10)
- net LIS3DH INT1: now also U2.11 (INT1)
- net LIS3DH INT2: now reaches U1.14 (GPIO11)
- net LIS3DH INT2: now also U2.9 (INT2)
- net I2C SDA: now reaches U1.15 (GPIO12)
- net I2C SCL: now reaches U1.16 (GPIO13)
- net LED MID: now reaches U1.17 (GPIO14)
- net LED MID: now also R23.1
- net at U1.2 (GPIO0): now also J3.1 (Pin_1)
- net at U1.26 (RUN): now also SW1.3 (K), SW1.4 (A)
- net BUTTON 1: now reaches U1.27 (GPIO16)
- net BUTTON 1: now also SW3.1, SW3.2
- net BUTTON 2: now reaches U1.28 (GPIO17)
- net BUTTON 2: now also SW4.1, SW4.2
- net LED S: now reaches U1.29 (GPIO18)
- net LED S: now also R15.1
- net at U1.3 (GPIO1): now also J3.3 (Pin_3)
- net LED SSE: now reaches U1.30 (GPIO19)
- net LED SSE: now also R19.1
- net LED SE: now reaches U1.31 (GPIO20)
- net LED SE: now also R16.1
- net LED ESE: now reaches U1.32 (GPIO21)
- net LED ESE: now also R20.1
- net LED E: now reaches U1.34 (GPIO22)
- net LED E: now also R17.1
- net LED ENE: now reaches U1.35 (GPIO23)
- net LED ENE: now also R21.1
- net LED NE: now reaches U1.36 (GPIO24)
- net LED NE: now also R18.1
- net LED NNE: now reaches U1.37 (GPIO25)
- net LED NNE: now also R22.1
- net LED N: now reaches U1.4 (GPIO2)
- net LED N: now also R5.1
- net TMP235 Out: now reaches U1.41 (GPIO29_ADC3)
- net TMP235 Out: now also C21.1, U6.3 (Vout)
- net LED NNW: now reaches U1.5 (GPIO3)
- net LED NNW: now also R7.1
- net LED NW: now reaches U1.6 (GPIO4)
- net LED NW: now also R9.1
- net LED WNW: now reaches U1.7 (GPIO5)
- net LED WNW: now also R10.1
- net LED W: now reaches U1.8 (GPIO6)
- net LED W: now also R11.1
- net LED WSW: now reaches U1.9 (GPIO7)
- net LED WSW: now also R13.1
- net at D2.2 (A): now also R7.2
- net at R5.2: now also D1.2 (A)
- new net: D13.2 (A), R19.2
- new net: D6.2 (A), R12.2
- new net: D14.2 (A), R20.2
- new net: D15.2 (A), R21.2
- new net: D11.2 (A), R17.2
- new net: D3.2 (A), R9.2
- new net: C22.1, R8.1, U6.4 (Vdd)
- new net: D4.2 (A), R10.2
- new net: D8.2 (A), R14.2
- new net: D17.2 (A), R23.2
- new net: D16.2 (A), R22.2
- new net: D12.2 (A), R18.2
- new net: D7.2 (A), R13.2
- new net: D9.2 (A), R15.2
- new net: D10.2 (A), R16.2
- new net: D5.2 (A), R11.2
- new net: JP1.2 (B), U2.7 (SDO)
- no-connect marks 0 -> 9
Other:
- note added: "Jumper selects USB to power the circuit, or battery"
- note removed: "Confirm Pinout and functionality with my Amazon board"
- moved on the sheet: C13, C14, C15, C16, C17, D1, D2, J2, J4, L1, R3, R4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
