File: Christmas Ornament 2024.kicad_sch (KiCad schematic)
At the start: 80 parts, among them J1 USB_B_Micro, J2 Conn_01x03, J3 Conn_01x03, J4 Conn_01x03, J5 Conn_01x03, SW1 PTS815, SW2 PTS815, SW3 PTS815, SW4 PTS815, U1 RP2040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

Commit message: PCB Layout beginning
Parts:
- R3: footprint Resistor_SMD:R_0805_2012Metric_Pad1.20x1.40mm_HandSolder -> Resistor_SMD:R_0402_1005Metric; JLCPCB PN C17436 -> C93945
- R4: footprint Resistor_SMD:R_0805_2012Metric_Pad1.20x1.40mm_HandSolder -> Resistor_SMD:R_0402_1005Metric; JLCPCB PN C17444 -> C25752
- Y1: footprint Crystal:Crystal_SMD_Abracon_ABM3-2Pin_5.0x3.2mm_HandSoldering -> Crystal:Crystal_SMD_Abracon_ABM3-2Pin_5.0x3.2mm
Connections:
- net +3V3: now also U1.1 (IOVDD), U1.10 (IOVDD), U1.22 (IOVDD), U1.33 (IOVDD), U1.42 (IOVDD), U1.43 (ADC_AVDD), U1.44 (VREG_IN), U1.48 (USB_VDD), U1.49 (IOVDD)
- net GND: no longer U1.1 (IOVDD), U1.10 (IOVDD), U1.22 (IOVDD), U1.33 (IOVDD), U1.42 (IOVDD), U1.43 (ADC_AVDD), U1.44 (VREG_IN), U1.48 (USB_VDD), U1.49 (IOVDD)
Changed lines of the file:
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@@
 	(paper "A4")
 	(junction
+		(at 111.76 45.72)
+		(diameter 0)
+		(color 0 0 0 0)
+	)
+	(junction
 		(at 33.02 142.24)
 		(diameter 0)
@@
 	)
 	(junction
-		(at 119.38 45.72)
+		(at 106.68 26.67)
 		(diameter 0)
 		(color 0 0 0 0)
 	)
 	(junction
-		(at 63.5 55.88)
+		(at 111.76 26.67)
 		(diameter 0)
 		(color 0 0 0 0)
 	)
 	(junction
-		(at 168.91 36.83)
+		(at 63.5 55.88)
 		(diameter 0)
 		(color 0 0 0 0)
 	)
 	(junction
-		(at 106.68 35.56)
+		(at 168.91 36.83)
 		(diameter 0)
 		(color 0 0 0 0)
@@
 	)
 	(junction
-		(at 119.38 36.83)
-		(diameter 0)
-		(color 0 0 0 0)
-	)
-	(junction
 		(at 128.27 26.67)
 		(diameter 0)
@@
 	)
 	(junction
+		(at 106.68 44.45)
+		(diameter 0)
+		(color 0 0 0 0)
+	)
+	(junction
 		(at 317.5 92.71)
 		(diameter 0)
@@
 		(color 0 0 0 0)
 	)
+	(junction
+		(at 119.38 26.67)
+		(diameter 0)
+		(color 0 0 0 0)
+	)
 	(no_connect
 		(at 281.94 33.02)
@@
 	(wire
 		(pts
-			(xy 320.04 38.1) (xy 320.04 40.64)
+			(xy 106.68 26.67) (xy 93.98 26.67)
 		)
 		(stroke
@@
 	(wire
 		(pts
-			(xy 48.26 132.08) (xy 48.26 129.54)
+			(xy 320.04 38.1) (xy 320.04 40.64)
 		)
 		(stroke
@@
 	(wire
 		(pts
-			(xy 361.95 163.83) (xy 364.49 163.83)
+			(xy 48.26 132.08) (xy 48.26 129.54)
 		)
 		(stroke
@@
 	(wire
 		(pts
-			(xy 128.27 24.13) (xy 128.27 26.67)
+			(xy 361.95 163.83) (xy 364.49 163.83)
 		)
 		(stroke
@@
 	(wire
 		(pts
+			(xy 111.76 26.67) (xy 119.38 26.67)
+		)
+		(stroke
+			(width 0)
+			(type default)
+		)
+	)
+	(wire
+		(pts
 			(xy 80.01 55.88) (xy 80.01 58.42)
 		)
@@
 	(wire
 		(pts
-			(xy 93.98 24.13) (xy 93.98 26.67)
+			(xy 106.68 24.13) (xy 106.68 26.67)
 		)
 		(stroke
@@
 	(wire
 		(pts
-			(xy 104.14 50.8) (xy 104.14 35.56)
+			(xy 104.14 50.8) (xy 104.14 44.45)
 		)
 		(stroke
@@
 	(wire
 		(pts
-			(xy 134.62 81.28) (xy 140.97 81.28)
+			(xy 106.68 26.67) (xy 106.68 44.45)
 		)
 		(stroke
@@
 	(wire
 		(pts
-			(xy 252.73 27.94) (xy 256.54 27.94)
+			(xy 134.62 81.28) (xy 140.97 81.28)
 		)
 		(stroke
@@
 	(wire
 		(pts
-			(xy 116.84 45.72) (xy 119.38 45.72)
+			(xy 252.73 27.94) (xy 256.54 27.94)
 		)
 		(stroke
@@
 	(wire
 		(pts
-			(xy 63.5 53.34) (xy 63.5 55.88)
+			(xy 116.84 45.72) (xy 119.38 45.72)
 		)
 		(stroke
@@
 	(wire
 		(pts
-			(xy 93.98 26.67) (xy 106.68 26.67)
+			(xy 63.5 53.34) (xy 63.5 55.88)
 		)
 		(stroke
@@
 	(wire
 		(pts
-			(xy 104.14 35.56) (xy 106.68 35.56)
+			(xy 104.14 44.45) (xy 106.68 44.45)
 		)
 		(stroke
@@
 	(wire
 		(pts
+			(xy 111.76 26.67) (xy 111.76 45.72)
+		)
+		(stroke
+			(width 0)
+			(type default)
+		)
+	)
+	(wire
+		(pts
 			(xy 45.72 24.13) (xy 45.72 21.59)
 		)
@@
 	(wire
 		(pts
+			(xy 106.68 44.45) (xy 106.68 50.8)
+		)
+		(stroke
+			(width 0)
+			(type default)
+		)
+	)
+	(wire
+		(pts
 			(xy 101.6 167.64) (xy 105.41 167.64)
 		)
@@
 	(wire
 		(pts
+			(xy 111.76 24.13) (xy 111.76 26.67)
+		)
+		(stroke
+			(width 0)
+			(type default)
+		)
+	)
+	(wire
+		(pts
 			(xy 149.86 60.96) (xy 149.86 58.42)
 		)
@@
 	(wire
 		(pts
-			(xy 106.68 35.56) (xy 106.68 50.8)
-		)
-		(stroke
-			(width 0)
-			(type default)
-		)
-	)
-	(wire
-		(pts
 			(xy 208.28 144.78) (xy 205.74 144.78)
 		)
@@
 	(wire
 		(pts
-			(xy 119.38 36.83) (xy 119.38 45.72)
-		)
-		(stroke
-			(width 0)
-			(type default)
-		)
-	)
-	(wire
-		(pts
 			(xy 31.75 127) (xy 33.02 127)
 		)
@@
 	(wire
 		(pts
-			(xy 106.68 26.67) (xy 106.68 35.56)
-		)
-		(stroke
-			(width 0)
-			(type default)
-		)
-	)
-	(wire
-		(pts
 			(xy 148.59 34.29) (xy 148.59 36.83)
 		)
@@
 	(symbol
 		(lib_id "power:+3V3")
-		(at 128.27 24.13 0)
+		(at 111.76 24.13 0)
 		(unit 1)
 		(exclude_from_sim no)
@@
 		(fields_autoplaced yes)
 		(property "Reference" "#PWR01"
-			(at 128.27 27.94 0)
+			(at 111.76 27.94 0)
 			(effects
 				(font
@@
 		)
 		(property "Value" "+3V3"
-			(at 128.27 19.05 0)
+			(at 111.76 19.05 0)
 			(effects
 				(font
@@
 		)
 		(property "Footprint" ""
-			(at 128.27 24.13 0)
+			(at 111.76 24.13 0)
 			(effects
 				(font
@@
 		)
 		(property "Datasheet" ""
-			(at 128.27 24.13 0)
+			(at 111.76 24.13 0)
 			(effects
 				(font
@@
 		)
 		(property "Description" "Power symbol creates a global label with name \"+3V3\""
-			(at 128.27 24.13 0)
+			(at 111.76 24.13 0)
 			(effects
 				(font
@@
 	(symbol
 		(lib_id "power:+1V1")
-		(at 93.98 24.13 0)
+		(at 106.68 24.13 0)
 		(unit 1)
 		(exclude_from_sim no)
@@
 		(fields_autoplaced yes)
 		(property "Reference" "#PWR02"
-			(at 93.98 27.94 0)
+			(at 106.68 27.94 0)
 			(effects
 				(font
@@
 		)
 		(property "Value" "+1V1"
-			(at 93.98 19.05 0)
+			(at 106.68 19.05 0)
 			(effects
 				(font
@@
 		)
 		(property "Footprint" ""
-			(at 93.98 24.13 0)
+			(at 106.68 24.13 0)
 			(effects
 				(font
@@
 		)
 		(property "Datasheet" ""
-			(at 93.98 24.13 0)
+			(at 106.68 24.13 0)
 			(effects
 				(font
@@
 		)
 		(property "Description" "Power symbol creates a global label with name \"+1V1\""
-			(at 93.98 24.13 0)
+			(at 106.68 24.13 0)
 			(effects
 				(font
@@
 			)
 		)
-		(property "Footprint" "Resistor_SMD:R_0805_2012Metric_Pad1.20x1.40mm_HandSolder"
+		(property "Footprint" "Resistor_SMD:R_0402_1005Metric"
 			(at 368.3 45.72 0)
 			(effects
@@
 			)
 		)
-		(property "JLCPCB PN" "C17436"
+		(property "JLCPCB PN" "C93945"
 			(at 368.3 45.72 0)
 			(effects
@@
 			)
 		)
-		(property "Footprint" "Resistor_SMD:R_0805_2012Metric_Pad1.20x1.40mm_HandSolder"
+		(property "Footprint" "Resistor_SMD:R_0402_1005Metric"
 			(at 368.3 54.61 0)
 			(effects
@@
 			)
 		)
-		(property "JLCPCB PN" "C17444"
+		(property "JLCPCB PN" "C25752"
 			(at 368.3 54.61 0)
 			(effects
@@
 			)
 		)
-		(property "Footprint" "Crystal:Crystal_SMD_Abracon_ABM3-2Pin_5.0x3.2mm_HandSoldering"
+		(property "Footprint" "Crystal:Crystal_SMD_Abracon_ABM3-2Pin_5.0x3.2mm"
 			(at 109.22 167.64 0)
 			(effects

Commit message: Layout in progress...
Parts:
- J2: footprint Connector_PinHeader_2.54mm:PinHeader_1x03_P2.54mm_Vertical -> Connector_JST:JST_SH_BM03B-SRSS-TB_1x03-1MP_P1.00mm_Vertical; JLCPCB PN DNP -> C160389
- J3: footprint Connector_PinHeader_2.54mm:PinHeader_1x03_P2.54mm_Vertical -> Connector_PinHeader_1.27mm:PinHeader_1x03_P1.27mm_Vertical
Changed lines of the file:
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@@
 			)
 		)
-		(property "Footprint" "Connector_PinHeader_2.54mm:PinHeader_1x03_P2.54mm_Vertical"
+		(property "Footprint" "Connector_JST:JST_SH_BM03B-SRSS-TB_1x03-1MP_P1.00mm_Vertical"
 			(at 24.13 110.49 0)
 			(effects
@@
 			)
 		)
-		(property "JLCPCB PN" "DNP"
+		(property "JLCPCB PN" "C160389"
 			(at 24.13 110.49 0)
 			(effects
@@
 			)
 		)
-		(property "Footprint" "Connector_PinHeader_2.54mm:PinHeader_1x03_P2.54mm_Vertical"
+		(property "Footprint" "Connector_PinHeader_1.27mm:PinHeader_1x03_P1.27mm_Vertical"
 			(at 160.02 55.88 0)
 			(effects

Commit message: PCB Layout and Routing complete
DRC
Parts:
- removed J3: Conn_01x03, Connector_PinHeader_1.27mm:PinHeader_1x03_P1.27mm_Vertical, symbol Connector_Generic:Conn_01x03
- added D18: Green LED, LED_SMD:LED_0805_2012Metric_Pad1.15x1.40mm_HandSolder, symbol Device:LED_Small
- added R24: 100, Resistor_SMD:R_0805_2012Metric_Pad1.20x1.40mm_HandSolder, symbol Device:R_Small
- J4: now not fitted; now left out of the parts list
- JP1: now left out of the parts list
Connections:
- net GND: now also D18.1 (K)
- net at U1.2 (GPIO0): now also R24.1
- new net: D18.2 (A), R24.2
- no-connect marks 9 -> 10
Other:
- note added: "Accelerometer"
- note added: "Boost Converter"
- note added: "Spirit Level LEDs"
- note added: "Temperature Sensor"
- note added: "User Inputs"
- note removed: "Confirm pinout"
- company: (none) -> Jacob Antoun
- title: (none) -> Christmas Ornament 2024
- moved on the sheet: C13, C14, C18, C19, C20, C3, D1, D10, D11, D12, D13, D14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
